File: hardware/sparkpunk.sch (EAGLE design)
At the start: 71 parts, among them IC1 556, IC2 CD4013B, IC3 LM358, IC4 LM358, J1 AUDIO-JACK2KIT

Commit message: Updates from prototype evaluation
Parts:
- added C10, C14, C15, C16: .1uf, SparkFun-Capacitors:CAPKIT
- added GATE: CV2, SparkFun-Connectors:M01SMDNS
- IC1: value 556 -> 7556
Connections:
- removed net N$7: IC1.CV, JP1.1
- removed net N$9: IC1.CV2, JP2.1
- removed net PTICH1: IC1.OUT, JP11.1, RV2.E, RV2.S
- new net VCC1: C10.1, IC1.CV2, JP2.1
- new net VCC2: C14.1, IC1.CV, JP1.1
- net FILT-OUT: now also IC3G2.OUT; no longer IC3G$2.OUT
- net GND: now also C10.2, C14.2, C15.2, C16.2, IC3G1.V-, IC4G1.V-; no longer IC3G$1.V-, IC4G$1.V-
- net N: now also IC4G1.+IN, IC4G2.+IN; no longer IC4G$1.+IN, IC4G$2.+IN
- net N$16: now also IC4G1.-IN, IC4G1.OUT; no longer IC4G$1.-IN, IC4G$1.OUT
- net N$25: now also IC4G2.-IN, IC4G2.OUT; no longer IC4G$2.-IN, IC4G$2.OUT
- net N$26: now also IC3G1.-IN; no longer IC3G$1.-IN
- net N$27: now also IC3G1.OUT, IC3G2.+IN; no longer IC3G$1.OUT, IC3G$2.+IN
- net N$31: now also IC3G2.-IN; no longer IC3G$2.-IN
- net N$4: now also GATE.1
- net PITCH1: now also IC1.OUT, JP11.1, RV2.E, RV2.S
- net VCC: now also C15.1, C16.1, IC3G1.V+, IC4G1.V+; no longer IC3G$1.V+, IC4G$1.V+
- net VREF: now also IC3G1.+IN; no longer IC3G$1.+IN
Other:
- note added: "Decoupling cap - place near IC1"
- note added: "Decoupling cap - place near IC2"
- note added: "V11"
- note removed: "V10"
- moved on the sheet: IC2A, IC2B, IC2P, JP1, JP2

Commit message: Updating sparkpunk parts with in-house ID#s
Parts:
- IC1: DIST digikey -> (none); DIST_ID ICM7556IPDZ-ND -> (none); PROD_ID (none) -> IC-11898
- R4, R5, R6, R7, R8: PROD_ID RES-09498 -> RES-10686
Changed lines of the file:
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@@
 <parts>
 <part name="IC1" library="SparkFun-AnalogIC" deviceset="556" device="KIT" value="7556">
-<attribute name="DIST" value="digikey"/>
-<attribute name="DIST_ID" value="ICM7556IPDZ-ND"/>
+<attribute name="PROD_ID" value="IC-11898"/>
 </part>
 <part name="RV3" library="SparkFun-Electromechanical" deviceset="POT" device="ALPS-KIT" value="10k">
@@
 </part>
 <part name="R4" library="SparkFun-Resistors" deviceset="RESISTOR" device="EZ" value="100k">
-<attribute name="PROD_ID" value="RES-09498"/>
+<attribute name="PROD_ID" value="RES-10686"/>
 </part>
 <part name="R5" library="SparkFun-Resistors" deviceset="RESISTOR" device="EZ" value="100k">
-<attribute name="PROD_ID" value="RES-09498"/>
+<attribute name="PROD_ID" value="RES-10686"/>
 </part>
 <part name="R6" library="SparkFun-Resistors" deviceset="RESISTOR" device="EZ" value="100k">
-<attribute name="PROD_ID" value="RES-09498"/>
+<attribute name="PROD_ID" value="RES-10686"/>
 </part>
 <part name="R7" library="SparkFun-Resistors" deviceset="RESISTOR" device="EZ" value="100k">
-<attribute name="PROD_ID" value="RES-09498"/>
+<attribute name="PROD_ID" value="RES-10686"/>
 </part>
 <part name="R8" library="SparkFun-Resistors" deviceset="RESISTOR" device="EZ" value="100k">
-<attribute name="PROD_ID" value="RES-09498"/>
+<attribute name="PROD_ID" value="RES-10686"/>
 </part>
 <part name="R9" library="SparkFun-Resistors" deviceset="RESISTOR" device="EZ" value="10k">
@@
 <instances>
 <instance part="IC1" gate="G$1" x="71.12" y="182.88">
-<attribute name="DIST" x="71.12" y="182.88" size="1.778" layer="96" display="off"/>
-<attribute name="DIST_ID" x="71.12" y="182.88" size="1.778" layer="96" display="off"/>
+<attribute name="PROD_ID" x="71.12" y="182.88" size="1.778" layer="96" display="off"/>
 </instance>
 <instance part="RV3" gate="G$1" x="114.3" y="182.88" rot="MR0">
@@
 <attribute name="PROD_ID" x="22.86" y="144.78" size="1.778" layer="96" rot="R180" display="off"/>
 </instance>
-<instance part="IC2" gate="A" x="50.8" y="66.04"/>
+<instance part="IC2" gate="A" x="50.8" y="66.04">
+<attribute name="PROD_ID" x="50.8" y="66.04" size="1.778" layer="96" display="off"/>
+</instance>
 <instance part="IC2" gate="B" x="50.8" y="30.48"/>
 <instance part="IC2" gate="P" x="93.98" y="63.5"/>

Commit message: One more sparkle part number.
Parts:
- D1: PROD_ID (none) -> DIO-11895
Changed lines of the file:
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@@
 <attribute name="DIST" value="sparkfun"/>
 <attribute name="DIST_ID" value="COM-10926"/>
+<attribute name="PROD_ID" value="DIO-11895"/>
 </part>
 <part name="SUPPLY1" library="SparkFun-Aesthetics" deviceset="VCC" device=""/>
@@
 <attribute name="DIST" x="353.06" y="106.68" size="1.778" layer="96" display="off"/>
 <attribute name="DIST_ID" x="353.06" y="106.68" size="1.778" layer="96" display="off"/>
+<attribute name="PROD_ID" x="353.06" y="106.68" size="1.778" layer="96" display="off"/>
 </instance>
 <instance part="SUPPLY1" gate="1" x="406.4" y="111.76"/>

Commit message: PCB update
Redesigned some aspects of PCB, for tighter integration with the
sequencer.
Parts:
- removed GATE: CV2, SparkFun-Connectors:M01SMDNS
- removed JP18: Vin, SparkFun-Connectors:M01SMDNS
- removed R15: 1Meg, SparkFun-Resistors:RESISTOREZ
- removed R16: 10k, SparkFun-Resistors:RESISTOREZ
- added D2: 1n4148, SparkFun-DiscreteSemi:DIODEKIT
- added D3: 1n5819, SparkFun-DiscreteSemi:DIODEPTH
- added S6: SPDT, SparkFun-Electromechanical:SWITCH-SPDTKIT
- C1: value .47uf -> .1uf; PROD_ID CAP-09152 -> CAP-08370
- C10, C14, C15: value .1uf -> 10uf/25V; device SparkFun-Capacitors:CAPKIT -> SparkFun-Capacitors:10UF-25V-20%(PTH)KIT; PROD_ID CAP-08370 -> (none)
- C12, C3: value 10uf/25V -> 1uf; device SparkFun-Capacitors:10UF-25V-20%(PTH)KIT -> SparkFun-Capacitors:CAPKIT; PROD_ID (none) -> CAP-09184
- C13: value 10uf/25V -> 1uf; device SparkFun-Capacitors:10UF-25V-20%(PTH)KIT -> SparkFun-Capacitors:CAPKIT; PROD_ID (none) -> CAP-9184
- C2: value 1uf -> .1uf; PROD_ID CAP-09184 -> CAP-08370
- C4: value 10uf/25V -> .47uf; device SparkFun-Capacitors:10UF-25V-20%(PTH)KIT -> SparkFun-Capacitors:CAPKIT; PROD_ID (none) -> CAP-09152
- C5: value 10uf/25V -> .1uf; device SparkFun-Capacitors:10UF-25V-20%(PTH)KIT -> SparkFun-Capacitors:CAPKIT; PROD_ID (none) -> CAP-08370
- C8: value 1uf -> 10uf/25V; device SparkFun-Capacitors:CAPKIT -> SparkFun-Capacitors:10UF-25V-20%(PTH)KIT; PROD_ID CAP-09184 -> (none)
- C9: value 1uf -> 10uf/25V; device SparkFun-Capacitors:CAPKIT -> SparkFun-Capacitors:10UF-25V-20%(PTH)KIT; PROD_ID CAP-9184 -> (none)
- D1: value 1n5819 -> 1n4148; device SparkFun-DiscreteSemi:DIODEPTH -> SparkFun-DiscreteSemi:DIODEKIT; DIST sparkfun -> (none); DIST_ID COM-10926 -> (none); PROD_ID DIO-11895 -> (none)
- JP11: value P1 -> P3
- JP12: value P1 -> P4
- JP13: value P2 -> P4
- JP14: value P2 -> SPK
- JP17: value Vsw -> GND
- JP3: value IN -> P1
- JP4: value CAP1 -> P1
- JP5: value S1 -> P2
- JP6: value S2 -> P2
- JP7: value P4 -> CAP1
- JP8: value P4 -> GATE
- JP9: value P3 -> IN
- R10, R9: value 10k -> 100k; PROD_ID RES-09435 -> RES-10686
- R11, R12: value 470 -> 10k; PROD_ID RES-10693 -> RES-09435
- R13: value 1k -> 10k; PROD_ID RES-08380 -> RES-09435
- R14: value 1Meg -> 1k; PROD_ID RES-09329 -> RES-08380
- R3: value 10k -> 470; PROD_ID RES-09435 -> RES-10693
- R4: value 100k -> 470; PROD_ID RES-10686 -> RES-10693
- R5: value 100k -> 1Meg; PROD_ID RES-10686 -> RES-09329
- RV1: device SparkFun-Electromechanical:POT_DUAL -> SparkFun-Electromechanical:POTALPS-KIT; DIST digikey -> (none); DIST_ID P2A5103-ND -> (none); PROD_ID (none) -> RES-09177
- RV3: device SparkFun-Electromechanical:POTALPS-KIT -> SparkFun-Electromechanical:POT_DUAL; DIST (none) -> digikey; DIST_ID (none) -> P2A5103-ND; PROD_ID RES-09177 -> (none)
Connections:
- removed net N$15: J1.RSH, JP6.1
- removed net N$6: R13.2, S5.C
- new net BUTTON: D1.A, S5.2, S5.A
- new net N$7: D3.A, S6.P
- new net N$9: R14.2, S5.C
- net FILT-OUT: now also JP13.1, RV3G$1.A; no longer JP7.1, RV1G$1.A
- net GND: now also C12.1, C13.2, C2.2, C3.1, C4.2, C5.2, JP17.1, R14.1, R5.2; no longer C10.2, C14.2, C15.2, C2.1, C8.1, C9.2, R10.1, R14.2, R15.2
- net N$1: now also D2.A, JP8.1; no longer D1.C, JP18.1, S5.2
- net N$12: now also JP4.1, R3.2, RV1.A; no longer JP12.1, R11.2, RV2.A
- net N$13: now also C10.-; no longer C3.-
- net N$14: now also JP14.1; no longer JP5.1
- net N$16: now also C14.+; no longer C13.+
- net N$17: now also C15.-; no longer C12.-
- net N$18: now also C10.+, R10.2; no longer C3.+, R7.2
- net N$19: now also C9.+, R9.2; no longer C4.+, R6.2
- net N$20: now also C9.-; no longer C4.-
- net N$21: now also C6.-, JP9.1; no longer C7.-, JP3.1
- net N$22: now also C6.+, R6.1; no longer C7.+, R8.1
- net N$23: now also C7.-; no longer C6.-
- net N$24: now also C8.-; no longer C5.-
- net N$25: now also C15.+; no longer C12.+
- net N$26: now also R10.1, R11.2, R6.2, R8.1, R9.1; no longer R3.2, R4.1, R5.1, R6.1, R8.2
- net N$27: now also R11.1; no longer R3.1
- net N$28: now also C8.+, R8.2; no longer C5.+, R5.2
- net N$29: now also C7.+, R7.2; no longer C6.+, R4.2
- net N$3: now also C4.1, R4.1; no longer C1.1, R12.1
- net N$30: now also C14.-; no longer C13.-
- net N$31: now also JP10.1, RV3G$2.E, RV3G$2.S; no longer JP9.1, RV1G$2.E, RV1G$2.S
- net N$33: now also C12.2, C13.1, JP11.1, JP12.1, RV3G$1.E, RV3G$1.S, RV3G$2.A; no longer C8.2, C9.1, JP10.1, JP8.1, RV1G$1.E, RV1G$1.S, RV1G$2.A
- net N$4: now also D1.C, D2.C, R5.1; no longer GATE.1, R14.1, R15.1, R16.1
- net N$8: now also JP6.1, R4.2, RV2.A; no longer JP14.1, R12.2, RV3.A
- net PITCH1: now also JP3.1, RV1.E, RV1.S; no longer JP11.1, RV2.E, RV2.S
- net PITCH2: now also JP5.1, RV2.E, RV2.S; no longer JP13.1, RV3.E, RV3.S
- net VBATT: now also S6.S; no longer D1.A
- net VCAP1: now also C3.2, JP7.1, R3.1; no longer C2.2, JP4.1, R11.1
- net VCC: now also C5.1, D3.C, R12.2; no longer C15.1, JP17.1, R16.2, R9.2, S5.A
- net VCC1: now also C2.1; no longer C10.1
- net VCC2: now also C1.1; no longer C14.1
- net VREF: now also R12.1, R13.2; no longer R10.2, R9.1
Other:
- note added: "Battery, Power Switch & Trigger"
- note added: "ON/OFF"
- note added: "V12"
- note removed: "Battery & Power Switch"
- note removed: "V11"
- moved on the sheet: BAT1, C1, C2, C6, C7, D1, JP10, JP11, JP12, JP13, JP14, JP16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

Commit message: Updated with feedback from beta builders.
Parts:
- BAT1: device SparkFun-Connectors:BC9VPC -> SparkFun-Connectors:BC9VPCKIT_SOLDERMASK
- D3: device SparkFun-DiscreteSemi:DIODEPTH -> SparkFun-DiscreteSemi:DIODE
Connections:
- removed net N$2: IC1.DIS, R1.1
- removed net N$5: IC1.DIS2, R2.1
- new net POT1: IC1.OUT, JP3.1, RV1.E, RV1.S
- new net POT2: IC1.OUT2, JP5.1, RV2.E, RV2.S
- net PITCH1: now also IC1.DIS, R1.1; no longer IC1.OUT, JP3.1, RV1.E, RV1.S
- net PITCH2: now also IC1.DIS2, R2.1; no longer IC1.OUT2, JP5.1, RV2.E, RV2.S
Other:
- note added: "V13"
- note removed: "V12"
