File: hardware/sparkpunk.brd (EAGLE design)
At the start: 88.9 x 68.6 mm, 75 parts, among them IC1 7556, IC2 CD4013B, IC3 LM358, IC4 LM358, J1 AUDIO-JACK2KIT

Commit message: Ready for Reds
Reviewed and ready to go.
Parts:
- moved LOGO2 2.62 mm to (33.7, 5.08)
- moved LOGO1 2.54 mm to (55.9, 3.81)
Other:
- board text added: "SOUND GENERATOR"
Changed lines of the file:
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@@
 <grid distance="0.05" unitdist="inch" unit="inch" style="lines" multiple="1" display="yes" altdistance="0.005" altunitdist="inch" altunit="inch"/>
 <layers>
-<layer number="1" name="Top" color="4" fill="1" visible="yes" active="yes"/>
+<layer number="1" name="Top" color="4" fill="1" visible="no" active="yes"/>
 <layer number="2" name="Route2" color="1" fill="3" visible="no" active="no"/>
 <layer number="3" name="Route3" color="4" fill="3" visible="no" active="no"/>
@@
 <layer number="14" name="Route14" color="1" fill="6" visible="no" active="no"/>
 <layer number="15" name="Route15" color="4" fill="6" visible="no" active="no"/>
-<layer number="16" name="Bottom" color="1" fill="1" visible="yes" active="yes"/>
+<layer number="16" name="Bottom" color="1" fill="1" visible="no" active="yes"/>
 <layer number="17" name="Pads" color="2" fill="1" visible="yes" active="yes"/>
 <layer number="18" name="Vias" color="2" fill="1" visible="yes" active="yes"/>
@@
 <layer number="20" name="Dimension" color="15" fill="1" visible="yes" active="yes"/>
 <layer number="21" name="tPlace" color="16" fill="1" visible="yes" active="yes"/>
-<layer number="22" name="bPlace" color="14" fill="1" visible="yes" active="yes"/>
+<layer number="22" name="bPlace" color="14" fill="1" visible="no" active="yes"/>
 <layer number="23" name="tOrigins" color="15" fill="1" visible="yes" active="yes"/>
 <layer number="24" name="bOrigins" color="15" fill="1" visible="yes" active="yes"/>
@@
 <layer number="49" name="Reference" color="7" fill="1" visible="no" active="yes"/>
 <layer number="50" name="dxf" color="7" fill="1" visible="no" active="no"/>
-<layer number="51" name="tDocu" color="6" fill="1" visible="yes" active="yes"/>
+<layer number="51" name="tDocu" color="6" fill="1" visible="no" active="yes"/>
 <layer number="52" name="bDocu" color="7" fill="1" visible="no" active="yes"/>
 <layer number="53" name="tGND_GNDA" color="7" fill="9" visible="no" active="no"/>
@@
 <wire x1="29.21" y1="61.595" x2="31.75" y2="61.595" width="0.254" layer="21"/>
 <wire x1="20.32" y1="60.96" x2="20.32" y2="68.58" width="0.254" layer="21"/>
+<text x="44.45" y="1.27" size="1.778" layer="21" font="vector" ratio="15" align="bottom-center">SOUND GENERATOR</text>
+<text x="44.45" y="1.27" size="1.778" layer="22" font="vector" ratio="15" rot="MR0" align="bottom-center">SOUND GENERATOR</text>
 </plain>
 <attributes>
@@
 </element>
 <element name="JP14" library="SparkFun-Connectors" package="1X01NS" value="SPK" x="69.85" y="67.31" rot="R90"/>
-<element name="LOGO1" library="SparkFun-Aesthetics" package="SFE_LOGO_NAME_FLAME_.2" value="SFE_LOGO_NAME_FLAME.2_INCH" x="55.88" y="1.27" rot="MR0"/>
+<element name="LOGO1" library="SparkFun-Aesthetics" package="SFE_LOGO_NAME_FLAME_.2" value="SFE_LOGO_NAME_FLAME.2_INCH" x="55.88" y="3.81" rot="MR0"/>
 <element name="LOGO3" library="SparkFun-Aesthetics" package="OSHW-LOGO-M" value="OSHW-LOGOM" x="6.35" y="34.29" rot="R90"/>
 <element name="LOGO4" library="SparkFun-Aesthetics" package="OSHW-LOGO-M" value="OSHW-LOGOM" x="60.325" y="5.715" rot="MR0"/>
@@
 <attribute name="PROD_ID" value="IC-11896" x="21.59" y="13.97" size="1.778" layer="27" rot="R270" display="off"/>
 </element>
-<element name="LOGO2" library="SparkFun-Aesthetics" package="SPARKPUNK_LOGO_.1" value="SPARKPUNK_LOGO.1INCH_TALL" x="33.02" y="2.54"/>
+<element name="LOGO2" library="SparkFun-Aesthetics" package="SPARKPUNK_LOGO_.1" value="SPARKPUNK_LOGO.1INCH_TALL" x="33.655" y="5.08"/>
 <element name="FRAME1" library="SparkFun-Aesthetics" package="CREATIVE_COMMONS" value="FRAME-LEDGER" x="24.13" y="-12.7"/>
 <element name="C5" library="SparkFun-Capacitors" package="CAP-PTH-SMALL-KIT" value=".1uf" x="25.4" y="60.96">
